File: cv-control.kicad_sch (KiCad schematic)
At the start: 55 parts, among them Q1 2N3904, Q2 2N3904, Q3 2N3904, Q4 2N3904, U4 TL074, U5 TL074

Commit message: Changes after tweaking
Parts:
- R21, R31: value 150k -> 220k
- R26, R29: value 2k -> 2k2
- R27, R28, R37: value 56k -> 100k
- R44, R45: value 100k -> 82k
Other:
- note added: "Output voltage range: -0.15v = short delay 0.0 = long delay 0.03 = glitching out"
- note removed: "Output voltage range: -0.16v = short delay 0.0 = long delay 0.03 = glitching out"
Changed lines of the file:
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@@
     (stroke (width 0) (type default) (color 0 0 0 0))
   )
-  (text "Output voltage range:\n-0.16v = short delay\n0.0 = long delay\n0.03 = glitching out"
+  (text "Output voltage range:\n-0.15v = short delay\n0.0 = long delay\n0.03 = glitching out"
     (at 200.66 31.75 0)
     (effects (font (size 1.27 1.27)) (justify left bottom))
@@
     (in_bom yes) (on_board yes)
     (property "Reference" "R29" (id 0) (at 198.12 105.2322 90))
-    (property "Value" "2k" (id 1) (at 198.12 107.5436 90))
+    (property "Value" "2k2" (id 1) (at 198.12 107.5436 90))
     (property "Footprint" "Rumblesan_Footprints:Resistor_THT_L6.3mm_D2.5mm_P10.16mm_Horizontal" (id 2) (at 198.12 108.712 90)
       (effects (font (size 1.27 1.27)) hide)
@@
     (in_bom yes) (on_board yes)
     (property "Reference" "R21" (id 0) (at 177.8 96.3422 90))
-    (property "Value" "150k" (id 1) (at 177.8 98.6536 90))
+    (property "Value" "220k" (id 1) (at 177.8 98.6536 90))
     (property "Footprint" "Rumblesan_Footprints:Resistor_THT_L6.3mm_D2.5mm_P10.16mm_Horizontal" (id 2) (at 177.8 99.822 90)
       (effects (font (size 1.27 1.27)) hide)
@@
     (in_bom yes) (on_board yes)
     (property "Reference" "R28" (id 0) (at 168.91 125.5522 90))
-    (property "Value" "56k" (id 1) (at 168.91 127.8636 90))
+    (property "Value" "100k" (id 1) (at 168.91 127.8636 90))
     (property "Footprint" "Rumblesan_Footprints:Resistor_THT_L6.3mm_D2.5mm_P10.16mm_Horizontal" (id 2) (at 168.91 129.032 90)
       (effects (font (size 1.27 1.27)) hide)
@@
     (in_bom yes) (on_board yes)
     (property "Reference" "R26" (id 0) (at 193.04 29.0322 90))
-    (property "Value" "2k" (id 1) (at 193.04 31.3436 90))
+    (property "Value" "2k2" (id 1) (at 193.04 31.3436 90))
     (property "Footprint" "Rumblesan_Footprints:Resistor_THT_L6.3mm_D2.5mm_P10.16mm_Horizontal" (id 2) (at 193.04 32.512 90)
       (effects (font (size 1.27 1.27)) hide)
@@
     (in_bom yes) (on_board yes)
     (property "Reference" "R44" (id 0) (at 86.36 32.8422 90))
-    (property "Value" "100k" (id 1) (at 86.36 35.1536 90))
+    (property "Value" "82k" (id 1) (at 86.36 35.1536 90))
     (property "Footprint" "Rumblesan_Footprints:Resistor_THT_L6.3mm_D2.5mm_P10.16mm_Horizontal" (id 2) (at 86.36 36.322 90)
       (effects (font (size 1.27 1.27)) hide)
@@
     (in_bom yes) (on_board yes)
     (property "Reference" "R27" (id 0) (at 175.26 49.3522 90))
-    (property "Value" "56k" (id 1) (at 175.26 51.6636 90))
+    (property "Value" "100k" (id 1) (at 175.26 51.6636 90))
     (property "Footprint" "Rumblesan_Footprints:Resistor_THT_L6.3mm_D2.5mm_P10.16mm_Horizontal" (id 2) (at 175.26 52.832 90)
       (effects (font (size 1.27 1.27)) hide)
@@
     (in_bom yes) (on_board yes)
     (property "Reference" "R45" (id 0) (at 86.36 110.3122 90))
-    (property "Value" "100k" (id 1) (at 86.36 112.6236 90))
+    (property "Value" "82k" (id 1) (at 86.36 112.6236 90))
     (property "Footprint" "Rumblesan_Footprints:Resistor_THT_L6.3mm_D2.5mm_P10.16mm_Horizontal" (id 2) (at 86.36 113.792 90)
       (effects (font (size 1.27 1.27)) hide)
@@
     (in_bom yes) (on_board yes)
     (property "Reference" "R37" (id 0) (at 181.61 87.4522 90))
-    (property "Value" "56k" (id 1) (at 181.61 89.7636 90))
+    (property "Value" "100k" (id 1) (at 181.61 89.7636 90))
     (property "Footprint" "Rumblesan_Footprints:Resistor_THT_L6.3mm_D2.5mm_P10.16mm_Horizontal" (id 2) (at 181.61 90.932 90)
       (effects (font (size 1.27 1.27)) hide)
@@
     (in_bom yes) (on_board yes)
     (property "Reference" "R31" (id 0) (at 172.72 17.6022 90))
-    (property "Value" "150k" (id 1) (at 172.72 19.9136 90))
+    (property "Value" "220k" (id 1) (at 172.72 19.9136 90))
     (property "Footprint" "Rumblesan_Footprints:Resistor_THT_L6.3mm_D2.5mm_P10.16mm_Horizontal" (id 2) (at 172.72 21.082 90)
       (effects (font (size 1.27 1.27)) hide)
