File: outputmix.kicad_sch (KiCad schematic)
At the start: 16 parts, among them U1 TL072

Commit message: Changes after tweaking
Parts:
- R2, R7: value 15k -> 10k
Changed lines of the file:
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@@
     (in_bom yes) (on_board yes)
     (property "Reference" "R7" (id 0) (at 119.38 106.5022 90))
-    (property "Value" "15k" (id 1) (at 119.38 108.8136 90))
+    (property "Value" "10k" (id 1) (at 119.38 108.8136 90))
     (property "Footprint" "Rumblesan_Footprints:Resistor_THT_L6.3mm_D2.5mm_P10.16mm_Horizontal" (id 2) (at 119.38 109.982 90)
       (effects (font (size 1.27 1.27)) hide)
@@
     (in_bom yes) (on_board yes)
     (property "Reference" "R2" (id 0) (at 125.5522 80.01 90))
-    (property "Value" "15k" (id 1) (at 127.8636 80.01 90))
+    (property "Value" "10k" (id 1) (at 127.8636 80.01 90))
     (property "Footprint" "Rumblesan_Footprints:Resistor_THT_L6.3mm_D2.5mm_P10.16mm_Horizontal" (id 2) (at 129.032 80.01 90)
       (effects (font (size 1.27 1.27)) hide)
